File: electronics/current_sensor_ldo/current_sensor_ldo.kicad_pcb (KiCad board)
At the start: 2 copper layers, 37.8 x 43.1 mm, 21 parts, among them J1 CS connector, J2 External connector, U1 ADP7104ARDZ-5.0-R7, U2 AD7685CRMZ, U3 ADP7104ARDZ-9.0-R7, U4 ADR435BRMZ, U5 INA253A3IPWR

Commit message: Update
Parts:
- moved C1 1.34 mm to (138.1, 93.0), turned to -90 degrees
- moved C6 1.16 mm to (138.3, 64.2), turned to -90 degrees
- moved U3 1.01 mm to (132.5, 64.5)
- moved C7 1.01 mm to (126.8, 64.3)
Routing:
- net /VIN: track 8.04 -> 68.1 mm
- net +9V: track 23.2 -> 24.2 mm
Other:
- board text added: "SDO"
