File: electronics/s3rvo_kicad/s3rvo.kicad_sch (KiCad schematic)
At the start: 44 parts, among them IC1 ADR4540BRZ, IC2 AD7685CRMZ, IC3 DRV8701P, J1 Conn_Enc, J2 Conn_CAN, Q1 CSD18540Q5B, Q2 CSD18540Q5B, Q3 CSD18540Q5B, Q4 CSD18540Q5B, SW1 SW_Push, U1 INA253A2IPWR, U2 STM32F446RCT6, U3 SN65HVD230, Y1 X322512MSB4SI

Commit message: update
Parts:
- removed C21: 220uF, Capacitor_SMD:CP_Elec_10x7.7, symbol Device:C_Polarized_Small
- removed C22, C24, C26: 1uF, Capacitor_SMD:C_0603_1608Metric, symbol Device:C_Small
- removed C23: 47uF, Capacitor_SMD:CP_Elec_10x7.7, symbol Device:C_Polarized_Small
- removed C25: 100nF, Capacitor_SMD:C_0603_1608Metric, symbol Device:C_Small
- removed IC1: ADR4540BRZ, Package_SO:SOIC-8_3.9x4.9mm_P1.27mm, symbol 0_servo:ADR4540BRZ
- removed IC3: DRV8701P, Package_DFN_QFN:VQFN-24-1EP_4x4mm_P0.5mm_EP2.45x2.45mm, symbol 1_motor:DRV8701P
- added C21, C23, C24: 1uF, PCM_Capacitor_SMD_AKL:C_0201_0603Metric, symbol PCM_Capacitor_AKL:C_0201
- added C22, C25: 100nF, PCM_Capacitor_SMD_AKL:C_0201_0603Metric, symbol PCM_Capacitor_AKL:C_0201
- added C26: 22uF, PCM_Capacitor_SMD_AKL:C_0201_0603Metric, symbol PCM_Capacitor_AKL:C_0201
- added C29: 1uF, Capacitor_SMD:C_0603_1608Metric, symbol Device:C_Small
- added C30, C33: 2.2uF, Capacitor_SMD:C_0603_1608Metric, symbol Device:C_Small
- added C31: 4.7uF, Capacitor_SMD:C_0603_1608Metric, symbol Device:C_Small
- added C32: 100nF, Capacitor_SMD:C_0402_1005Metric, symbol Device:C_Small
- added C34: 22uF, Capacitor_SMD:C_0603_1608Metric, symbol Device:C_Small
- added D1: SS210, Diode_SMD:D_SMA, symbol Diode:SS210
- added IC1: ADR4550BRZ, Package_SO:SOIC-8_3.9x4.9mm_P1.27mm, symbol 0_servo:ADR4550BRZ
- added IC3: DRV8703QRHBRQ1, Package_DFN_QFN:QFN-32-1EP_5x5mm_P0.5mm_EP3.45x3.45mm_ThermalVias, symbol 0_servo:DRV8703QRHBRQ1
- added IC4: MP2459GJ-Z, Package_TO_SOT_SMD:TSOT-23-6, symbol 0_servo:MP2459GJ-Z
- added L2: 10uH, Inductor_SMD:L_Coilcraft_LPS5030, symbol Device:L_Small
- added R2, R3: 10k, Resistor_SMD:R_0402_1005Metric, symbol Device:R_Small
- added R4: 576k, Resistor_SMD:R_0402_1005Metric, symbol Device:R_Small
- added R5: 100k, Resistor_SMD:R_0402_1005Metric, symbol Device:R_Small
- added U4: XC6206P332MR-G, Package_TO_SOT_SMD:SOT-23-3, symbol Regulator_Linear:XC6206PxxxMR
- added U8: ADP7142AUJZ-5.0, Package_TO_SOT_SMD:TSOT-23-5, symbol Regulator_Linear:ADP7142AUJZ-5.0
- C19: value 10uF -> 22uF
- C27: value 0.1uF -> 1uF
Connections:
- net DVDD is gone; now on net +3V3: R1.1
- net GND_D is gone; now on net nFAULT: R1.2
- net GND_M is gone; now on net GND: C27.2, Q2.1 (S), Q2.2 (S), Q2.3 (S), Q4.1 (S), Q4.2 (S), Q4.3 (S)
- net +3V3: now also C29.1, R2.1, R3.1, U4.2 (VO)
- net +5V: now also C33.1, IC1.2 (IN), U8.4 (SENSE/ADJ), U8.5 (VOUT)
- net AVDD: now also C24.1, IC3.14 (AVDD), IC3.15 (VREF)
- net CS_M: now also U1.1 (IS-); no longer U1.1,2,3 (IS-)
- net CS_P: now also U1.18 (IS+); no longer U1.18,19,20 (IS+)
- net GND: now also U1.15 (GND), U1.6 (GND), C23.2, C24.2, C25.2, C26.2, C29.2, C30.2, C31.2, C33.2, C34.2, D1.2 (A), IC1.4 (GND), IC3.1 (GND), IC3.13 (GND), IC3.17 (GND), IC3.21 (SP), IC3.22 (SN), IC3.23 (SL2), IC4.2 (GND), R4.2, U4.1 (GND), U8.2 (GND); no longer U1.6,15 (GND)
- net IN1: now also IC3.2 (IN1/PH)
- net IN2: now also IC3.3 (IN2/EN)
- net VM: now also C21.1, C25.1, C26.1, C31.1, IC3.27 (VDRAIN), IC3.28 (VM), IC4.5 (VIN); no longer C27.1
- net nFAULT: now also IC3.10 (nFAULT)
- net nSLEEP: now also IC3.8 (nSLEEP)
- net at C13.1, C15.1: now also IC1.6 (OUT)
- net GH1: no longer names the net of Q1.4 (G)
- net GH1: now also IC3.18 (GH1)
- net GH2: no longer names the net of Q3.4 (G)
- net GH2: now also IC3.26 (GH2)
- net GL1: no longer names the net of Q2.4 (G)
- net GL1: now also IC3.20 (GL1)
- net GL2: no longer names the net of Q4.4 (G)
- net GL2: now also IC3.24 (GL2)
- net M_A: no longer names the net of Q1.1 (S), Q1.2 (S), Q1.3 (S), Q2.5 (D)
- net M_A: now also IC3.19 (SH1)
- net M_B: no longer names the net of Q3.1 (S), Q3.2 (S), Q3.3 (S), Q4.5 (D)
- net M_B: now also IC3.25 (SH2)
- new net: C21.2, IC3.29 (VCP)
- new net: C22.1, IC3.30 (CPH)
- new net: C22.2, IC3.31 (CPL)
- new net: C23.1, IC3.12 (DVDD)
- new net +5V5: C27.1, C30.1, C34.1, L2.2, R5.1, U4.3 (VI), U8.1 (VIN), U8.3 (EN)
- new net BST: C32.1, IC4.1 (BST)
- new net FB: IC4.3 (FB), R4.1, R5.2
- new net MODE: IC3.11 (MODE)
- new net SCLK: IC3.7 (SCLK)
- new net SDI: IC3.6 (SDI)
- new net SDO: IC3.4 (SDO), R3.2
- new net SW: C32.2, D1.1 (K), IC4.6 (SW), L2.1
- new net nSCS: IC3.5 (nSCS)
- new net nWDFLT: IC3.9 (nWDFLT), R2.2
- no-connect marks 3 -> 2
Other:
- note added: "Package_DFN_QFN:QFN-32-1EP_5x5mm_P0.5mm_EP3.45x3.45mm_ThermalVias"
- moved on the sheet: Q1, Q2, Q3, Q4, U1

Commit message: Update
Parts:
- renumbered C31 to C19, C19 to C20, C32 to C21, C20 to C22, C34 to C23, C30 to C24, C27 to C25, C29 to C26, C33 to C27, C23 to C29, C25 to C30, C24 to C31, C26 to C32, C21 to C33, C22 to C34, U1 to IC2, U2 to IC3, IC2 to IC5, U8 to IC6, U4 to IC7, U3 to IC8, IC3 to IC9, Q3 to Q1, Q4 to Q2, Q1 to Q3, Q2 to Q4, R5 to R1, R4 to R2, R2 to R4, R1 to R5
Connections:
- net +3V3: now also J2.1 (Pin_1)
- net +5V: no longer J2.1 (Pin_1)
- net CS_M: now also IC9.25 (SH2), Q1.1 (S), Q1.2 (S), Q1.3 (S), Q2.5 (D)
- net CS_P: now also IC9.19 (SH1), Q3.1 (S), Q3.2 (S), Q3.3 (S), Q4.5 (D)
- net V_REF: now also C13.1, C15.1, IC1.6 (OUT)
